File: pcb/psu-30w.kicad_pcb (KiCad board)
At the start: 2 copper layers, 200 x 81 mm, 43 parts, among them J1 Barrel_Jack, J18 Power Switch Option, U1 R-78E5.0-1.0

Commit message: Wärmefallen und KICAD 6
Other:
- net class Default removed
- net class PWR removed
